File: Quadsense.sch (KiCad schematic (older format))
At the start: 49 parts, among them IC1 BME280, IC2 AP7330, IC3 ADC_LTC2497, IC4 BME280, P1 CONN_6, P2 CONN_6, P3 CONN_6, P4 CONN_6, P5 CONN_8, Q1 AO3418

Commit message: Saved changes
Parts:
- LOGO1: footprint (none) -> Logo:Logo
Changed lines of the file:
@@
 $EndComp
 $Comp
-L GND #PWR7
+L GND #PWR01
 U 1 1 5C6461C4
 P 4900 2550
-F 0 "#PWR7" H 4925 2600 50  0001 C CNN
+F 0 "#PWR01" H 4925 2600 50  0001 C CNN
 F 1 "GND" H 4900 2400 50  0000 C CNN
 F 2 "" H 4900 2550 60  0000 C CNN
@@
 $EndComp
 $Comp
-L 5V #PWR6
+L 5V #PWR02
 U 1 1 5C6461DA
 P 3800 1750
-F 0 "#PWR6" H 3825 1700 60  0001 C CNN
+F 0 "#PWR02" H 3825 1700 60  0001 C CNN
 F 1 "5V" H 3800 1900 50  0000 C CNN
 F 2 "" H 3800 1750 60  0000 C CNN
@@
 $EndComp
 $Comp
-L GND #PWR10
+L GND #PWR03
 U 1 1 5C6480D4
 P 5800 6850
-F 0 "#PWR10" H 5825 6900 50  0001 C CNN
+F 0 "#PWR03" H 5825 6900 50  0001 C CNN
 F 1 "GND" H 5800 6700 50  0000 C CNN
 F 2 "" H 5800 6850 60  0000 C CNN
@@
 $EndComp
 $Comp
-L 3V3 #PWR15
+L 3V3 #PWR04
 U 1 1 5C6545DA
 P 9700 1750
-F 0 "#PWR15" H 9725 1700 60  0001 C CNN
+F 0 "#PWR04" H 9725 1700 60  0001 C CNN
 F 1 "3V3" H 9700 1900 50  0000 C CNN
 F 2 "" H 9700 1750 60  0000 C CNN
@@
 $EndComp
 $Comp
-L GND #PWR16
+L GND #PWR05
 U 1 1 5C65462E
 P 9700 2400
-F 0 "#PWR16" H 9725 2450 50  0001 C CNN
+F 0 "#PWR05" H 9725 2450 50  0001 C CNN
 F 1 "GND" H 9700 2250 50  0000 C CNN
 F 2 "" H 9700 2400 60  0000 C CNN
@@
 $EndComp
 $Comp
-L 3V3 #PWR13
+L 3V3 #PWR06
 U 1 1 5C654F38
 P 8250 1750
-F 0 "#PWR13" H 8275 1700 60  0001 C CNN
+F 0 "#PWR06" H 8275 1700 60  0001 C CNN
 F 1 "3V3" H 8250 1900 50  0000 C CNN
 F 2 "" H 8250 1750 60  0000 C CNN
@@
 3V3\n5V\nGND\nID1\nSCL\nID2\nSDA\nEN
 $Comp
-L GND #PWR3
+L GND #PWR07
 U 1 1 5C6F1ACC
 P 1650 2600
-F 0 "#PWR3" H 1675 2650 50  0001 C CNN
+F 0 "#PWR07" H 1675 2650 50  0001 C CNN
 F 1 "GND" H 1650 2450 50  0000 C CNN
 F 2 "" H 1650 2600 60  0000 C CNN
@@
 $EndComp
 $Comp
-L 3V3 #PWR4
+L 3V3 #PWR08
 U 1 1 5C6F1B4C
 P 1700 1550
-F 0 "#PWR4" H 1725 1500 60  0001 C CNN
+F 0 "#PWR08" H 1725 1500 60  0001 C CNN
 F 1 "3V3" H 1700 1700 50  0000 C CNN
 F 2 "" H 1700 1550 60  0000 C CNN
@@
 $EndComp
 $Comp
-L 5V #PWR1
+L 5V #PWR09
 U 1 1 5C6F1BCC
 P 1550 1550
-F 0 "#PWR1" H 1575 1500 60  0001 C CNN
+F 0 "#PWR09" H 1575 1500 60  0001 C CNN
 F 1 "5V" H 1550 1700 50  0000 C CNN
 F 2 "" H 1550 1550 60  0000 C CNN
@@
 $EndComp
 $Comp
-L GND #PWR5
+L GND #PWR010
 U 1 1 5C6F649C
 P 1950 7250
-F 0 "#PWR5" H 1975 7300 50  0001 C CNN
+F 0 "#PWR010" H 1975 7300 50  0001 C CNN
 F 1 "GND" H 1950 7100 50  0000 C CNN
 F 2 "" H 1950 7250 60  0000 C CNN
@@
 	8300 2100 8150 2100
 $Comp
-L PWR_FLAG #FLAG4
+L PWR_FLAG #FLAG011
 U 1 1 5C6FD365
 P 7050 1650
-F 0 "#FLAG4" H 7050 1750 50  0001 C CNN
+F 0 "#FLAG011" H 7050 1750 50  0001 C CNN
 F 1 "PWR_FLAG" H 7050 1850 50  0000 C CNN
 F 2 "" H 7050 1650 60  0000 C CNN
@@
 	7050 1850 7050 1650
 $Comp
-L PWR_FLAG #FLAG1
+L PWR_FLAG #FLAG012
 U 1 1 5C6FD994
 P 1400 1500
-F 0 "#FLAG1" H 1400 1600 50  0001 C CNN
+F 0 "#FLAG012" H 1400 1600 50  0001 C CNN
 F 1 "PWR_FLAG" H 1400 1700 50  0000 C CNN
 F 2 "" H 1400 1500 60  0000 C CNN
@@
 $EndComp
 $Comp
-L PWR_FLAG #FLAG2
+L PWR_FLAG #FLAG013
 U 1 1 5C6FDA3C
 P 1850 2650
-F 0 "#FLAG2" H 1850 2750 50  0001 C CNN
+F 0 "#FLAG013" H 1850 2750 50  0001 C CNN
 F 1 "PWR_FLAG" H 1850 2850 50  0000 C CNN
 F 2 "" H 1850 2650 60  0000 C CNN
@@
 Connection ~ 5300 5950
 $Comp
-L 4V #PWR9
+L 4V #PWR014
 U 1 1 5C706294
 P 5800 1750
-F 0 "#PWR9" H 5825 1700 60  0001 C CNN
+F 0 "#PWR014" H 5825 1700 60  0001 C CNN
 F 1 "4V" H 5800 1900 50  0000 C CNN
 F 2 "" H 5800 1750 60  0000 C CNN
@@
 $EndComp
 $Comp
-L A4V #PWR12
+L A4V #PWR015
 U 1 1 5C70635C
 P 6850 1750
-F 0 "#PWR12" H 6875 1700 60  0001 C CNN
+F 0 "#PWR015" H 6875 1700 60  0001 C CNN
 F 1 "A4V" H 6850 1900 50  0000 C CNN
 F 2 "" H 6850 1750 60  0000 C CNN
@@
 $EndComp
 $Comp
-L A4V #PWR8
+L A4V #PWR016
 U 1 1 5C706C1D
 P 5300 4400
-F 0 "#PWR8" H 5325 4350 60  0001 C CNN
+F 0 "#PWR016" H 5325 4350 60  0001 C CNN
 F 1 "A4V" H 5300 4550 50  0000 C CNN
 F 2 "" H 5300 4400 60  0000 C CNN
@@
 $EndComp
 $Comp
-L 4V #PWR11
+L 4V #PWR017
 U 1 1 5C706CE5
 P 6250 4400
-F 0 "#PWR11" H 6275 4350 60  0001 C CNN
+F 0 "#PWR017" H 6275 4350 60  0001 C CNN
 F 1 "4V" H 6250 4550 50  0000 C CNN
 F 2 "" H 6250 4400 60  0000 C CNN
@@
 $EndComp
 $Comp
-L A4V #PWR2
+L A4V #PWR018
 U 1 1 5C706F15
 P 1550 3850
-F 0 "#PWR2" H 1575 3800 60  0001 C CNN
+F 0 "#PWR018" H 1575 3800 60  0001 C CNN
 F 1 "A4V" H 1550 4000 50  0000 C CNN
 F 2 "" H 1550 3850 60  0000 C CNN
@@
 $EndComp
 $Comp
-L PWR_FLAG #FLAG3
+L PWR_FLAG #FLAG019
 U 1 1 5C76DA5F
 P 1900 1500
-F 0 "#FLAG3" H 1900 1600 50  0001 C CNN
+F 0 "#FLAG019" H 1900 1600 50  0001 C CNN
 F 1 "PWR_FLAG" H 1900 1700 50  0000 C CNN
 F 2 "" H 1900 1500 60  0000 C CNN
@@
 $EndComp
 $Comp
-L 3V3 #PWR17
+L 3V3 #PWR020
 U 1 1 5CEE62EE
 P 9700 2900
-F 0 "#PWR17" H 9725 2850 60  0001 C CNN
+F 0 "#PWR020" H 9725 2850 60  0001 C CNN
 F 1 "3V3" H 9700 3050 50  0000 C CNN
 F 2 "" H 9700 2900 60  0000 C CNN
@@
 $EndComp
 $Comp
-L GND #PWR18
+L GND #PWR021
 U 1 1 5CEE62F4
 P 9700 3500
-F 0 "#PWR18" H 9725 3550 50  0001 C CNN
+F 0 "#PWR021" H 9725 3550 50  0001 C CNN
 F 1 "GND" H 9700 3350 50  0000 C CNN
 F 2 "" H 9700 3500 60  0000 C CNN
@@
 $EndComp
 $Comp
-L 3V3 #PWR14
+L 3V3 #PWR022
 U 1 1 5CEE62FA
 P 8250 2900
-F 0 "#PWR14" H 8275 2850 60  0001 C CNN
+F 0 "#PWR022" H 8275 2850 60  0001 C CNN
 F 1 "3V3" H 8250 3050 50  0000 C CNN
 F 2 "" H 8250 2900 60  0000 C CNN
@@
 F 0 "LOGO1" H 9400 6050 60  0000 C CNN
 F 1 "Logo" H 9400 6250 60  0000 C CNN
-F 2 "" H 9400 6300 60  0001 C CNN
+F 2 "Logo:Logo" H 9400 6300 60  0001 C CNN
 F 3 "" H 9400 6300 60  0001 C CNN
 	1    9400 6150
